File: anavi-rtc-3032.kicad_pcb (KiCad board)
At the start: 2 copper layers, 21.5 x 25 mm, 12 parts, among them J1 Conn_01x06_Pin

Commit message: Adjust silkscreen labels
Adjust the silkscreen labels becase KEYSTONE 3000 battery holder
supports multiple size, most notably CR1216 and CR1220.

Signed-off-by: Leon Anavi <leon@anavi.org>
Parts:
- CR1216/CR1220 Battery: renamed from CR1216 Battery
Changed lines of the file:
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@@
 			(drillshape 0)
 			(scaleselection 1)
-			(outputdirectory "plots/anavi-rtc-3032-r10a/")
+			(outputdirectory "plots/anavi-rtc-3032-r10b/")
 		)
 	)
@@
 		(descr "http://www.keyelco.com/product-pdf.cfm?p=777")
 		(tags "Keystone type 3000 coin cell retainer")
-		(property "Reference" "CR1216 Battery"
+		(property "Reference" "CR1216/CR1220 Battery"
 			(at 0 8.575 90)
 			(layer "B.SilkS")
